File: src/windF12.kicad_pcb (KiCad board)
At the start: 2 copper layers, 267.8 x 21 mm, 25 parts, among them SW1 SW_Push_45deg, SW10 SW_Push_45deg, SW11 SW_Push_45deg, SW12 SW_Push_45deg, SW2 SW_Push_45deg, SW3 SW_Push_45deg, SW4 SW_Push_45deg, SW5 SW_Push_45deg, SW6 SW_Push_45deg, SW7 SW_Push_45deg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

Commit message: stuff
Parts:
- added D13: LED_SK6812MINI, ScottoKeebs_Components:LED_SK6812MINI, B.Cu at (24.6, 32.6)
- added D14: LED_SK6812MINI, ScottoKeebs_Components:LED_SK6812MINI, B.Cu at (43.8, 32.4)
- added D15: LED_SK6812MINI, ScottoKeebs_Components:LED_SK6812MINI, B.Cu at (62.8, 32.4)
- added D16: LED_SK6812MINI, ScottoKeebs_Components:LED_SK6812MINI, B.Cu at (81.8, 32.4)
- added D17: LED_SK6812MINI, ScottoKeebs_Components:LED_SK6812MINI, B.Cu at (119.8, 32.4)
- added D18: LED_SK6812MINI, ScottoKeebs_Components:LED_SK6812MINI, B.Cu at (138.6, 32.4)
- added D19: LED_SK6812MINI, ScottoKeebs_Components:LED_SK6812MINI, B.Cu at (157.8, 32.4)
- added D20: LED_SK6812MINI, ScottoKeebs_Components:LED_SK6812MINI, B.Cu at (176.8, 32.4)
- added D21: LED_SK6812MINI, ScottoKeebs_Components:LED_SK6812MINI, B.Cu at (214.7, 32.6)
- added D22: LED_SK6812MINI, ScottoKeebs_Components:LED_SK6812MINI, B.Cu at (233.7, 32.8)
- added D23: LED_SK6812MINI, ScottoKeebs_Components:LED_SK6812MINI, B.Cu at (252.7, 32.6)
- added D24: LED_SK6812MINI, ScottoKeebs_Components:LED_SK6812MINI, B.Cu at (271.7, 32.5)
Connections:
- U1 pad 8: unconnected-(U1-P1.12_RX_D7-Pad8) -> led
Routing:
- net +5V: track 0.00 -> 280.7 mm, vias 0 -> 1
- net GND: track 0.00 -> 272.7 mm, vias 0 -> 18
- net Net-(D16-DOUT): track 0.00 -> 33.3 mm
- net Net-(D20-DOUT): track 0.00 -> 33.2 mm
- net Net-(D13-DOUT): track 0.00 -> 14.4 mm
- net Net-(D18-DOUT): track 0.00 -> 14.4 mm
- net Net-(D21-DOUT): track 0.00 -> 14.3 mm
- net Net-(D14-DOUT): track 0.00 -> 14.2 mm
- net Net-(D19-DOUT): track 0.00 -> 14.2 mm
- net Net-(D15-DOUT): track 0.00 -> 14.2 mm
- net Net-(D22-DOUT): track 0.00 -> 14.2 mm
- net Net-(D23-DOUT): track 0.00 -> 14.1 mm
- net Net-(D17-DOUT): track 0.00 -> 14.0 mm
- net led: track 0.00 -> 5.83 mm
- net c3: track 246.6 -> 248.0 mm
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