File: src/windF12.kicad_pcb (KiCad board)
At the start: 2 copper layers, 267.8 x 21 mm, 37 parts, among them SW1 SW_Push_45deg, SW10 SW_Push_45deg, SW11 SW_Push_45deg, SW12 SW_Push_45deg, SW2 SW_Push_45deg, SW3 SW_Push_45deg, SW4 SW_Push_45deg, SW5 SW_Push_45deg, SW6 SW_Push_45deg, SW7 SW_Push_45deg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

Commit message: w
Parts:
- added H1: MountingHole_Pad, MountingHole:MountingHole_2.2mm_M2_Pad, F.Cu at (111.8, 43.2)
- added H2: MountingHole_Pad, MountingHole:MountingHole_2.2mm_M2_Pad, F.Cu at (207.0, 43.2)
- moved D24 258.9 mm to (32.2, 130.9), turned to 180 degrees
- moved D23 239.6 mm to (32.2, 126.3), turned to 180 degrees
- moved D22 220.2 mm to (32.2, 121.7), turned to 180 degrees
- moved D21 201.1 mm to (32.2, 117.1), turned to 180 degrees
- moved D20 165.2 mm to (32.4, 112.5), turned to 180 degrees
- moved D19 146.4 mm to (32.4, 107.9), turned to 180 degrees
- moved D18 127.7 mm to (32.4, 103.3), turned to 180 degrees
- moved D17 109.7 mm to (32.4, 98.7), turned to 180 degrees
- moved D16 78.9 mm to (32.2, 93.7), turned to 180 degrees
- moved D15 62.6 mm to (31.3, 86.5), turned to 180 degrees
- moved D9 19.0 mm to (217.8, 43.1)
- moved SW11 19.0 mm to (266.7, 38.1)
- moved SW12 19.0 mm to (285.8, 38.1)
- moved SW10 19.0 mm to (247.7, 38.1)
- moved SW9 18.9 mm to (228.6, 38.1)
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Routing:
- net +5V: track 280.7 -> 0.00 mm, vias 1 -> 0
- net GND: track 272.7 -> 0.00 mm, vias 18 -> 0
- net c4: track 262.0 -> 0.00 mm
- net c3: track 248.0 -> 0.00 mm
- net r3: track 246.4 -> 0.00 mm
- net c2: track 223.2 -> 0.00 mm
- net c1: track 201.7 -> 0.00 mm
- net r2: track 144.6 -> 0.00 mm, vias 1 -> 0
- net r1: track 50.5 -> 0.00 mm
- net Net-(D16-DOUT): track 33.3 -> 0.00 mm
- net Net-(D20-DOUT): track 33.2 -> 0.00 mm
- net Net-(D1-A): track 15.1 -> 0.00 mm
- net Net-(D13-DOUT): track 14.4 -> 0.00 mm
- net Net-(D18-DOUT): track 14.4 -> 0.00 mm
- net Net-(D21-DOUT): track 14.3 -> 0.00 mm
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Other:
- board size 267.8 x 21 mm -> 268.9 x 21.2 mm
- board text added: "2025"
- board text added: "Made by Vejas"
- board text removed: "Made by Vejas 2025"

Commit message: loads
Parts:
- moved D24 264.5 mm to (283.2, 47.6), turned to 0 degrees
- moved D23 244.9 mm to (264.2, 47.6), turned to 0 degrees
- moved D22 225.4 mm to (245.1, 47.6), turned to 0 degrees
- moved D21 205.9 mm to (226.1, 47.6), turned to 0 degrees
- moved D20 168.6 mm to (188.0, 47.6), turned to 0 degrees
- moved D19 149.3 mm to (168.9, 47.6), turned to 0 degrees
- moved D18 130.0 mm to (149.9, 47.6), turned to 0 degrees
- moved D17 110.8 mm to (130.7, 47.6), turned to 0 degrees
- moved D16 76.1 mm to (92.7, 47.6), turned to 0 degrees
- moved D15 57.5 mm to (73.7, 47.6), turned to 0 degrees
Routing:
- net GND: track 0.00 -> 286.2 mm, vias 0 -> 13
- net +5V: track 0.00 -> 280.7 mm, vias 0 -> 1
- net c4: track 0.00 -> 272.8 mm
- net r3: track 0.00 -> 246.2 mm
- net c3: track 0.00 -> 238.3 mm, vias 0 -> 8
- net c2: track 0.00 -> 215.5 mm, vias 0 -> 10
- net c1: track 0.00 -> 202.3 mm, vias 0 -> 12
- net r2: track 0.00 -> 142.5 mm, vias 0 -> 1
- net r1: track 0.00 -> 51.2 mm
- net Net-(D20-DOUT): track 0.00 -> 33.3 mm
- net Net-(D16-DOUT): track 0.00 -> 33.2 mm
- net Net-(D1-A): track 0.00 -> 15.3 mm
- net Net-(D17-DOUT): track 0.00 -> 14.4 mm
- net Net-(D21-DOUT): track 0.00 -> 14.3 mm
- net Net-(D18-DOUT): track 0.00 -> 14.3 mm
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